File: hardware/piavr.kicad_sch (KiCad schematic)
At the start: 6 parts, among them J1 GPIO, U1 CAT24C256

Commit message: added hardware chips
Other:
- added sheet DAC (DAC.kicad_sch)
- added sheet DSP (DSP.kicad_sch)
- added sheet eARC (eARC.kicad_sch)
- note removed: "Additional pin functions: https://pinout.xyz/"
